Commit message: Removed build files

File: robot_ws/src/robot_description/urdf/assem.xacro (robot description, xacro)
@@ -12,5 +12,5 @@
     <origin xyz="0 0 0" rpy="0 0 0"/>
     <geometry>
-      <mesh filename="package://robot_description/meshes/base_link.stl" scale="0.001 0.001 0.001"/>
+      <mesh filename="file://$(find robot_description)/meshes/base_link.stl" scale="0.001 0.001 0.001"/>
     </geometry>
     <material name="steel_satin"/>
@@ -19,5 +19,5 @@
     <origin xyz="0 0 0" rpy="0 0 0"/>
     <geometry>
-      <mesh filename="package://robot_description/meshes/base_link.stl" scale="0.001 0.001 0.001"/>
+      <mesh filename="file://$(find robot_description)/meshes/base_link.stl" scale="0.001 0.001 0.001"/>
     </geometry>
   </collision>
@@ -35,5 +35,5 @@
     <origin xyz="-0.1184 -0.076 -0.0196" rpy="0 0 0"/>
     <geometry>
-      <mesh filename="package://robot_description/meshes/Right_Front_Leg_Mount_v1_1.stl" scale="0.001 0.001 0.001"/>
+      <mesh filename="file://$(find robot_description)/meshes/Right_Front_Leg_Mount_v1_1.stl" scale="0.001 0.001 0.001"/>
     </geometry>
     <material name="steel_satin"/>
@@ -42,5 +42,5 @@
     <origin xyz="-0.1184 -0.076 -0.0196" rpy="0 0 0"/>
     <geometry>
-      <mesh filename="package://robot_description/meshes/Right_Front_Leg_Mount_v1_1.stl" scale="0.001 0.001 0.001"/>
+      <mesh filename="file://$(find robot_description)/meshes/Right_Front_Leg_Mount_v1_1.stl" scale="0.001 0.001 0.001"/>
     </geometry>
   </collision>
@@ -55,5 +55,5 @@
     <origin xyz="0.1184 -0.076 -0.0196" rpy="0 0 0"/>
     <geometry>
-      <mesh filename="package://robot_description/meshes/Right_Back_Leg_Mount_v1_1.stl" scale="0.001 0.001 0.001"/>
+      <mesh filename="file://$(find robot_description)/meshes/Right_Back_Leg_Mount_v1_1.stl" scale="0.001 0.001 0.001"/>
     </geometry>
     <material name="steel_satin"/>
@@ -62,5 +62,5 @@
     <origin xyz="0.1184 -0.076 -0.0196" rpy="0 0 0"/>
     <geometry>
-      <mesh filename="package://robot_description/meshes/Right_Back_Leg_Mount_v1_1.stl" scale="0.001 0.001 0.001"/>
+      <mesh filename="file://$(find robot_description)/meshes/Right_Back_Leg_Mount_v1_1.stl" scale="0.001 0.001 0.001"/>
     </geometry>
   </collision>
@@ -75,5 +75,5 @@
     <origin xyz="0.1184 0.076 -0.0196" rpy="0 0 0"/>
     <geometry>
-      <mesh filename="package://robot_description/meshes/Left_Back_Leg_Mount_v1_1.stl" scale="0.001 0.001 0.001"/>
+      <mesh filename="file://$(find robot_description)/meshes/Left_Back_Leg_Mount_v1_1.stl" scale="0.001 0.001 0.001"/>
     </geometry>
     <material name="steel_satin"/>
@@ -82,5 +82,5 @@
     <origin xyz="0.1184 0.076 -0.0196" rpy="0 0 0"/>
     <geometry>
-      <mesh filename="package://robot_description/meshes/Left_Back_Leg_Mount_v1_1.stl" scale="0.001 0.001 0.001"/>
+      <mesh filename="file://$(find robot_description)/meshes/Left_Back_Leg_Mount_v1_1.stl" scale="0.001 0.001 0.001"/>
     </geometry>
   </collision>
@@ -95,5 +95,5 @@
     <origin xyz="-0.1184 0.076 -0.0196" rpy="0 0 0"/>
     <geometry>
-      <mesh filename="package://robot_description/meshes/Left_Front_Leg_Mount_v1_1.stl" scale="0.001 0.001 0.001"/>
+      <mesh filename="file://$(find robot_description)/meshes/Left_Front_Leg_Mount_v1_1.stl" scale="0.001 0.001 0.001"/>
     </geometry>
     <material name="steel_satin"/>
@@ -102,5 +102,5 @@
     <origin xyz="-0.1184 0.076 -0.0196" rpy="0 0 0"/>
     <geometry>
-      <mesh filename="package://robot_description/meshes/Left_Front_Leg_Mount_v1_1.stl" scale="0.001 0.001 0.001"/>
+      <mesh filename="file://$(find robot_description)/meshes/Left_Front_Leg_Mount_v1_1.stl" scale="0.001 0.001 0.001"/>
     </geometry>
   </collision>
@@ -115,5 +115,5 @@
     <origin xyz="-0.164597 -0.103749 -0.038258" rpy="0 0 0"/>
     <geometry>
-      <mesh filename="package://robot_description/meshes/Servo_Horn_v3_1.stl" scale="0.001 0.001 0.001"/>
+      <mesh filename="file://$(find robot_description)/meshes/Servo_Horn_v3_1.stl" scale="0.001 0.001 0.001"/>
     </geometry>
     <material name="steel_satin"/>
@@ -122,5 +122,5 @@
     <origin xyz="-0.164597 -0.103749 -0.038258" rpy="0 0 0"/>
     <geometry>
-      <mesh filename="package://robot_description/meshes/Servo_Horn_v3_1.stl" scale="0.001 0.001 0.001"/>
+      <mesh filename="file://$(find robot_description)/meshes/Servo_Horn_v3_1.stl" scale="0.001 0.001 0.001"/>
     </geometry>
   </collision>
@@ -135,5 +135,5 @@
     <origin xyz="-0.143947 -0.103749 -0.017258" rpy="0 0 0"/>
     <geometry>
-      <mesh filename="package://robot_description/meshes/Servo_Horn_v3_2.stl" scale="0.001 0.001 0.001"/>
+      <mesh filename="file://$(find robot_description)/meshes/Servo_Horn_v3_2.stl" scale="0.001 0.001 0.001"/>
     </geometry>
     <material name="steel_satin"/>
@@ -142,5 +142,5 @@
     <origin xyz="-0.143947 -0.103749 -0.017258" rpy="0 0 0"/>
     <geometry>
-      <mesh filename="package://robot_description/meshes/Servo_Horn_v3_2.stl" scale="0.001 0.001 0.001"/>
+      <mesh filename="file://$(find robot_description)/meshes/Servo_Horn_v3_2.stl" scale="0.001 0.001 0.001"/>
     </geometry>
   </collision>
@@ -155,5 +155,5 @@
     <origin xyz="0.144387 -0.103775 -0.038162" rpy="0 0 0"/>
     <geometry>
-      <mesh filename="package://robot_description/meshes/Servo_Horn_v3_4.stl" scale="0.001 0.001 0.001"/>
+      <mesh filename="file://$(find robot_description)/meshes/Servo_Horn_v3_4.stl" scale="0.001 0.001 0.001"/>
     </geometry>
     <material name="steel_satin"/>
@@ -162,5 +162,5 @@
     <origin xyz="0.144387 -0.103775 -0.038162" rpy="0 0 0"/>
     <geometry>
-      <mesh filename="package://robot_description/meshes/Servo_Horn_v3_4.stl" scale="0.001 0.001 0.001"/>
+      <mesh filename="file://$(find robot_description)/meshes/Servo_Horn_v3_4.stl" scale="0.001 0.001 0.001"/>
     </geometry>
   </collision>
@@ -175,5 +175,5 @@
     <origin xyz="0.164387 -0.103775 -0.017162" rpy="0 0 0"/>
     <geometry>
-      <mesh filename="package://robot_description/meshes/Servo_Horn_v3_3.stl" scale="0.001 0.001 0.001"/>
+      <mesh filename="file://$(find robot_description)/meshes/Servo_Horn_v3_3.stl" scale="0.001 0.001 0.001"/>
     </geometry>
     <material name="steel_satin"/>
@@ -182,5 +182,5 @@
     <origin xyz="0.164387 -0.103775 -0.017162" rpy="0 0 0"/>
     <geometry>
-      <mesh filename="package://robot_description/meshes/Servo_Horn_v3_3.stl" scale="0.001 0.001 0.001"/>
+      <mesh filename="file://$(find robot_description)/meshes/Servo_Horn_v3_3.stl" scale="0.001 0.001 0.001"/>
     </geometry>
   </collision>
@@ -195,5 +195,5 @@
     <origin xyz="-0.164597 0.103749 -0.038258" rpy="0 0 0"/>
     <geometry>
-      <mesh filename="package://robot_description/meshes/Servo_Horn_v3_5.stl" scale="0.001 0.001 0.001"/>
+      <mesh filename="file://$(find robot_description)/meshes/Servo_Horn_v3_5.stl" scale="0.001 0.001 0.001"/>
     </geometry>
     <material name="steel_satin"/>
@@ -202,5 +202,5 @@
     <origin xyz="-0.164597 0.103749 -0.038258" rpy="0 0 0"/>
     <geometry>
-      <mesh filename="package://robot_description/meshes/Servo_Horn_v3_5.stl" scale="0.001 0.001 0.001"/>
+      <mesh filename="file://$(find robot_description)/meshes/Servo_Horn_v3_5.stl" scale="0.001 0.001 0.001"/>
     </geometry>
   </collision>
@@ -215,5 +215,5 @@
     <origin xyz="-0.143947 0.103749 -0.017258" rpy="0 0 0"/>
     <geometry>
-      <mesh filename="package://robot_description/meshes/Servo_Horn_v3_8.stl" scale="0.001 0.001 0.001"/>
+      <mesh filename="file://$(find robot_description)/meshes/Servo_Horn_v3_8.stl" scale="0.001 0.001 0.001"/>
     </geometry>
     <material name="steel_satin"/>
@@ -222,5 +222,5 @@
     <origin xyz="-0.143947 0.103749 -0.017258" rpy="0 0 0"/>
     <geometry>
-      <mesh filename="package://robot_description/meshes/Servo_Horn_v3_8.stl" scale="0.001 0.001 0.001"/>
+      <mesh filename="file://$(find robot_description)/meshes/Servo_Horn_v3_8.stl" scale="0.001 0.001 0.001"/>
     </geometry>
   </collision>
@@ -235,5 +235,5 @@
     <origin xyz="0.144387 0.103775 -0.038162" rpy="0 0 0"/>
     <geometry>
-      <mesh filename="package://robot_description/meshes/Servo_Horn_v3_7.stl" scale="0.001 0.001 0.001"/>
+      <mesh filename="file://$(find robot_description)/meshes/Servo_Horn_v3_7.stl" scale="0.001 0.001 0.001"/>
     </geometry>
     <material name="steel_satin"/>
@@ -242,5 +242,5 @@
     <origin xyz="0.144387 0.103775 -0.038162" rpy="0 0 0"/>
     <geometry>
-      <mesh filename="package://robot_description/meshes/Servo_Horn_v3_7.stl" scale="0.001 0.001 0.001"/>
+      <mesh filename="file://$(find robot_description)/meshes/Servo_Horn_v3_7.stl" scale="0.001 0.001 0.001"/>
     </geometry>
   </collision>
@@ -255,5 +255,5 @@
     <origin xyz="0.164387 0.103775 -0.017162" rpy="0 0 0"/>
     <geometry>
-      <mesh filename="package://robot_description/meshes/Servo_Horn_v3_6.stl" scale="0.001 0.001 0.001"/>
+      <mesh filename="file://$(find robot_description)/meshes/Servo_Horn_v3_6.stl" scale="0.001 0.001 0.001"/>
     </geometry>
     <material name="steel_satin"/>
@@ -262,5 +262,5 @@
     <origin xyz="0.164387 0.103775 -0.017162" rpy="0 0 0"/>
     <geometry>
-      <mesh filename="package://robot_description/meshes/Servo_Horn_v3_6.stl" scale="0.001 0.001 0.001"/>
+      <mesh filename="file://$(find robot_description)/meshes/Servo_Horn_v3_6.stl" scale="0.001 0.001 0.001"/>
     </geometry>
   </collision>
@@ -275,5 +275,5 @@
     <origin xyz="0.165037 -0.115355 -0.017162" rpy="0 0 0"/>
     <geometry>
-      <mesh filename="package://robot_description/meshes/Left_Link_v4_1.stl" scale="0.001 0.001 0.001"/>
+      <mesh filename="file://$(find robot_description)/meshes/Left_Link_v4_1.stl" scale="0.001 0.001 0.001"/>
     </geometry>
     <material name="steel_satin"/>
@@ -282,5 +282,5 @@
     <origin xyz="0.165037 -0.115355 -0.017162" rpy="0 0 0"/>
     <geometry>
-      <mesh filename="package://robot_description/meshes/Left_Link_v4_1.stl" scale="0.001 0.001 0.001"/>
+      <mesh filename="file://$(find robot_description)/meshes/Left_Link_v4_1.stl" scale="0.001 0.001 0.001"/>
     </geometry>
   </collision>
@@ -295,5 +295,5 @@
     <origin xyz="0.099908 -0.115355 0.06636" rpy="0 0 0"/>
     <geometry>
-      <mesh filename="package://robot_description/meshes/Foot_v3_1.stl" scale="0.001 0.001 0.001"/>
+      <mesh filename="file://$(find robot_description)/meshes/Foot_v3_1.stl" scale="0.001 0.001 0.001"/>
     </geometry>
     <material name="steel_satin"/>
@@ -302,5 +302,5 @@
     <origin xyz="0.099908 -0.115355 0.06636" rpy="0 0 0"/>
     <geometry>
-      <mesh filename="package://robot_description/meshes/Foot_v3_1.stl" scale="0.001 0.001 0.001"/>
+      <mesh filename="file://$(find robot_description)/meshes/Foot_v3_1.stl" scale="0.001 0.001 0.001"/>
     </geometry>
   </collision>
@@ -315,5 +315,5 @@
     <origin xyz="-0.143797 -0.115329 -0.017258" rpy="0 0 0"/>
     <geometry>
-      <mesh filename="package://robot_description/meshes/Left_Link_v4_2.stl" scale="0.001 0.001 0.001"/>
+      <mesh filename="file://$(find robot_description)/meshes/Left_Link_v4_2.stl" scale="0.001 0.001 0.001"/>
     </geometry>
     <material name="steel_satin"/>
@@ -322,5 +322,5 @@
     <origin xyz="-0.143797 -0.115329 -0.017258" rpy="0 0 0"/>
     <geometry>
-      <mesh filename="package://robot_description/meshes/Left_Link_v4_2.stl" scale="0.001 0.001 0.001"/>
+      <mesh filename="file://$(find robot_description)/meshes/Left_Link_v4_2.stl" scale="0.001 0.001 0.001"/>
     </geometry>
   </collision>
