Commit message: Added ros2 control + some reorg

File: robot_ws/src/robot_description/urdf/assem.xacro (robot description, xacro)
@@ -1,765 +1,6 @@
 <?xml version="1.0" ?>
 <robot name="assem" xmlns:xacro="http://www.ros.org/wiki/xacro">
-<xacro:include filename="$(find robot_description)/urdf/materials.xacro" />
-<xacro:include filename="$(find robot_description)/urdf/assem.trans" />
-<link name="base_link">
-  <inertial>
-    <origin xyz="-0.008382264142625067 -1.4798434925308436e-05 0.030113658418836745" rpy="0 0 0"/>
-    <mass value="10.123728045116188"/>
-    <inertia ixx="0.03254" iyy="0.280159" izz="0.3037" ixy="-3.1e-05" iyz="-1e-06" ixz="0.001839"/>
-  </inertial>
-  <visual>
-    <origin xyz="0 0 0" rpy="0 0 0"/>
-    <geometry>
-      <mesh filename="file://$(find robot_description)/meshes/base_link.stl" scale="0.001 0.001 0.001"/>
-    </geometry>
-    <material name="steel_satin"/>
-  </visual>
-  <collision>
-    <origin xyz="0 0 0" rpy="0 0 0"/>
-    <geometry>
-      <mesh filename="file://$(find robot_description)/meshes/base_link.stl" scale="0.001 0.001 0.001"/>
-    </geometry>
-  </collision>
-</link>
-<link name="Right_Front_Leg_Mount_v1_1">
-  <inertial>
-    <origin xyz="0.03322621293445238 0.004607470996659868 0.011279980581351271" rpy="0 0 0"/>
-    <mass value="0.791396210786452"/>
-    <inertia ixx="0.000288" iyy="0.000453" izz="0.000409" ixy="1.4e-05" iyz="-6e-06" ixz="-6e-06"/>
-  </inertial>
-  <visual>
-    <origin xyz="-0.1184 -0.076 -0.0196" rpy="0 0 0"/>
-    <geometry>
-      <mesh filename="file://$(find robot_description)/meshes/Right_Front_Leg_Mount_v1_1.stl" scale="0.001 0.001 0.001"/>
-    </geometry>
-    <material name="steel_satin"/>
-  </visual>
-  <collision>
-    <origin xyz="-0.1184 -0.076 -0.0196" rpy="0 0 0"/>
-    <geometry>
-      <mesh filename="file://$(find robot_description)/meshes/Right_Front_Leg_Mount_v1_1.stl" scale="0.001 0.001 0.001"/>
-    </geometry>
-  </collision>
-</link>
-<link name="Right_Back_Leg_Mount_v1_1">
-  <inertial>
-    <origin xyz="-0.03453360704195005 0.004633032360894143 0.011213744397462203" rpy="0 0 0"/>
-    <mass value="0.7913962107864516"/>
-    <inertia ixx="0.000288" iyy="0.000458" izz="0.000413" ixy="1.2e-05" iyz="-6e-06" ixz="8e-06"/>
-  </inertial>
-  <visual>
-    <origin xyz="0.1184 -0.076 -0.0196" rpy="0 0 0"/>
-    <geometry>
-      <mesh filename="file://$(find robot_description)/meshes/Right_Back_Leg_Mount_v1_1.stl" scale="0.001 0.001 0.001"/>
-    </geometry>
-    <material name="steel_satin"/>
-  </visual>
-  <collision>
-    <origin xyz="0.1184 -0.076 -0.0196" rpy="0 0 0"/>
-    <geometry>
-      <mesh filename="file://$(find robot_description)/meshes/Right_Back_Leg_Mount_v1_1.stl" scale="0.001 0.001 0.001"/>
-    </geometry>
-  </collision>
-</link>
-<link name="Left_Back_Leg_Mount_v1_1">
-  <inertial>
-    <origin xyz="-0.03453360706419445 -0.004633032653077587 0.011213744349241432" rpy="0 0 0"/>
-    <mass value="0.7913962228945977"/>
-    <inertia ixx="0.000288" iyy="0.000458" izz="0.000413" ixy="-1.2e-05" iyz="6e-06" ixz="8e-06"/>
-  </inertial>
-  <visual>
-    <origin xyz="0.1184 0.076 -0.0196" rpy="0 0 0"/>
-    <geometry>
-      <mesh filename="file://$(find robot_description)/meshes/Left_Back_Leg_Mount_v1_1.stl" scale="0.001 0.001 0.001"/>
-    </geometry>
-    <material name="steel_satin"/>
-  </visual>
-  <collision>
-    <origin xyz="0.1184 0.076 -0.0196" rpy="0 0 0"/>
-    <geometry>
-      <mesh filename="file://$(find robot_description)/meshes/Left_Back_Leg_Mount_v1_1.stl" scale="0.001 0.001 0.001"/>
-    </geometry>
-  </collision>
-</link>
-<link name="Left_Front_Leg_Mount_v1_1">
-  <inertial>
-    <origin xyz="0.033226212974938135 -0.004607471288838219 0.011279980533589536" rpy="0 0 0"/>
-    <mass value="0.791396222894598"/>
-    <inertia ixx="0.000288" iyy="0.000453" izz="0.000409" ixy="-1.4e-05" iyz="6e-06" ixz="-6e-06"/>
-  </inertial>
-  <visual>
-    <origin xyz="-0.1184 0.076 -0.0196" rpy="0 0 0"/>
-    <geometry>
-      <mesh filename="file://$(find robot_description)/meshes/Left_Front_Leg_Mount_v1_1.stl" scale="0.001 0.001 0.001"/>
-    </geometry>
-    <material name="steel_satin"/>
-  </visual>
-  <collision>
-    <origin xyz="-0.1184 0.076 -0.0196" rpy="0 0 0"/>
-    <geometry>
-      <mesh filename="file://$(find robot_description)/meshes/Left_Front_Leg_Mount_v1_1.stl" scale="0.001 0.001 0.001"/>
-    </geometry>
-  </collision>
-</link>
-<link name="Servo_Horn_v3_1">
-  <inertial>
-    <origin xyz="0.00849626146165297 -2.908683761748687e-05 -1.6025929275784168e-06" rpy="0 0 0"/>
-    <mass value="0.010282942996218928"/>
-    <inertia ixx="1e-06" iyy="1e-06" izz="1e-06" ixy="-0.0" iyz="0.0" ixz="0.0"/>
-  </inertial>
-  <visual>
-    <origin xyz="-0.164597 -0.103749 -0.038258" rpy="0 0 0"/>
-    <geometry>
-      <mesh filename="file://$(find robot_description)/meshes/Servo_Horn_v3_1.stl" scale="0.001 0.001 0.001"/>
-    </geometry>
-    <material name="steel_satin"/>
-  </visual>
-  <collision>
-    <origin xyz="-0.164597 -0.103749 -0.038258" rpy="0 0 0"/>
-    <geometry>
-      <mesh filename="file://$(find robot_description)/meshes/Servo_Horn_v3_1.stl" scale="0.001 0.001 0.001"/>
-    </geometry>
-  </collision>
-</link>
-<link name="Servo_Horn_v3_2">
-  <inertial>
-    <origin xyz="-0.008496002222424276 -2.9086837616723593e-05 1.9981492505212473e-06" rpy="0 0 0"/>
-    <mass value="0.010282942996218928"/>
-    <inertia ixx="1e-06" iyy="1e-06" izz="1e-06" ixy="0.0" iyz="-0.0" ixz="0.0"/>
-  </inertial>
-  <visual>
-    <origin xyz="-0.143947 -0.103749 -0.017258" rpy="0 0 0"/>
-    <geometry>
-      <mesh filename="file://$(find robot_description)/meshes/Servo_Horn_v3_2.stl" scale="0.001 0.001 0.001"/>
-    </geometry>
-    <material name="steel_satin"/>
-  </visual>
-  <collision>
-    <origin xyz="-0.143947 -0.103749 -0.017258" rpy="0 0 0"/>
-    <geometry>
-      <mesh filename="file://$(find robot_description)/meshes/Servo_Horn_v3_2.stl" scale="0.001 0.001 0.001"/>
-    </geometry>
-  </collision>
-</link>
-<link name="Servo_Horn_v3_4">
-  <inertial>
-    <origin xyz="0.008495912831059382 -2.9238910956921882e-05 -1.8426360164636169e-06" rpy="0 0 0"/>
-    <mass value="0.010282942996218928"/>
-    <inertia ixx="1e-06" iyy="1e-06" izz="1e-06" ixy="-0.0" iyz="0.0" ixz="0.0"/>
-  </inertial>
-  <visual>
-    <origin xyz="0.144387 -0.103775 -0.038162" rpy="0 0 0"/>
-    <geometry>
-      <mesh filename="file://$(find robot_description)/meshes/Servo_Horn_v3_4.stl" scale="0.001 0.001 0.001"/>
-    </geometry>
-    <material name="steel_satin"/>
-  </visual>
-  <collision>
-    <origin xyz="0.144387 -0.103775 -0.038162" rpy="0 0 0"/>
-    <geometry>
-      <mesh filename="file://$(find robot_description)/meshes/Servo_Horn_v3_4.stl" scale="0.001 0.001 0.001"/>
-    </geometry>
-  </collision>
-</link>
-<link name="Servo_Horn_v3_3">
-  <inertial>
-    <origin xyz="-0.008496349973848794 -2.923891095629738e-05 1.7582700742799218e-06" rpy="0 0 0"/>
-    <mass value="0.010282942996218928"/>
-    <inertia ixx="1e-06" iyy="1e-06" izz="1e-06" ixy="0.0" iyz="-0.0" ixz="0.0"/>
-  </inertial>
-  <visual>
-    <origin xyz="0.164387 -0.103775 -0.017162" rpy="0 0 0"/>
-    <geometry>
-      <mesh filename="file://$(find robot_description)/meshes/Servo_Horn_v3_3.stl" scale="0.001 0.001 0.001"/>
-    </geometry>
-    <material name="steel_satin"/>
-  </visual>
-  <collision>
-    <origin xyz="0.164387 -0.103775 -0.017162" rpy="0 0 0"/>
-    <geometry>
-      <mesh filename="file://$(find robot_description)/meshes/Servo_Horn_v3_3.stl" scale="0.001 0.001 0.001"/>
-    </geometry>
-  </collision>
-</link>
-<link name="Servo_Horn_v3_5">
-  <inertial>
-    <origin xyz="0.008496261461652804 2.9086837618014227e-05 1.998089645890988e-06" rpy="0 0 0"/>
-    <mass value="0.010282942996218928"/>
-    <inertia ixx="1e-06" iyy="1e-06" izz="1e-06" ixy="0.0" iyz="0.0" ixz="-0.0"/>
-  </inertial>
-  <visual>
-    <origin xyz="-0.164597 0.103749 -0.038258" rpy="0 0 0"/>
-    <geometry>
-      <mesh filename="file://$(find robot_description)/meshes/Servo_Horn_v3_5.stl" scale="0.001 0.001 0.001"/>
-    </geometry>
-    <material name="steel_satin"/>
-  </visual>
-  <collision>
-    <origin xyz="-0.164597 0.103749 -0.038258" rpy="0 0 0"/>
-    <geometry>
-      <mesh filename="file://$(find robot_description)/meshes/Servo_Horn_v3_5.stl" scale="0.001 0.001 0.001"/>
-    </geometry>
-  </collision>
-</link>
-<link name="Servo_Horn_v3_8">
-  <inertial>
-    <origin xyz="-0.008496002222424415 2.9086837617570138e-05 -1.602533322913463e-06" rpy="0 0 0"/>
-    <mass value="0.010282942996218928"/>
-    <inertia ixx="1e-06" iyy="1e-06" izz="1e-06" ixy="-0.0" iyz="-0.0" ixz="-0.0"/>
-  </inertial>
-  <visual>
-    <origin xyz="-0.143947 0.103749 -0.017258" rpy="0 0 0"/>
-    <geometry>
-      <mesh filename="file://$(find robot_description)/meshes/Servo_Horn_v3_8.stl" scale="0.001 0.001 0.001"/>
-    </geometry>
-    <material name="steel_satin"/>
-  </visual>
-  <collision>
-    <origin xyz="-0.143947 0.103749 -0.017258" rpy="0 0 0"/>
-    <geometry>
-      <mesh filename="file://$(find robot_description)/meshes/Servo_Horn_v3_8.stl" scale="0.001 0.001 0.001"/>
-    </geometry>
-  </collision>
-</link>
-<link name="Servo_Horn_v3_7">
-  <inertial>
-    <origin xyz="0.008495912831059105 2.923891095736597e-05 1.7580465570474213e-06" rpy="0 0 0"/>
-    <mass value="0.010282942996218928"/>
-    <inertia ixx="1e-06" iyy="1e-06" izz="1e-06" ixy="0.0" iyz="0.0" ixz="-0.0"/>
-  </inertial>
-  <visual>
-    <origin xyz="0.144387 0.103775 -0.038162" rpy="0 0 0"/>
-    <geometry>
-      <mesh filename="file://$(find robot_description)/meshes/Servo_Horn_v3_7.stl" scale="0.001 0.001 0.001"/>
-    </geometry>
-    <material name="steel_satin"/>
-  </visual>
-  <collision>
-    <origin xyz="0.144387 0.103775 -0.038162" rpy="0 0 0"/>
-    <geometry>
-      <mesh filename="file://$(find robot_description)/meshes/Servo_Horn_v3_7.stl" scale="0.001 0.001 0.001"/>
-    </geometry>
-  </collision>
-</link>
-<link name="Servo_Horn_v3_6">
-  <inertial>
-    <origin xyz="-0.008496349973849043 2.923891095668596e-05 -1.8424124992970359e-06" rpy="0 0 0"/>
-    <mass value="0.010282942996218928"/>
-    <inertia ixx="1e-06" iyy="1e-06" izz="1e-06" ixy="-0.0" iyz="-0.0" ixz="-0.0"/>
-  </inertial>
-  <visual>
-    <origin xyz="0.164387 0.103775 -0.017162" rpy="0 0 0"/>
-    <geometry>
-      <mesh filename="file://$(find robot_description)/meshes/Servo_Horn_v3_6.stl" scale="0.001 0.001 0.001"/>
-    </geometry>
-    <material name="steel_satin"/>
-  </visual>
-  <collision>
-    <origin xyz="0.164387 0.103775 -0.017162" rpy="0 0 0"/>
-    <geometry>
-      <mesh filename="file://$(find robot_description)/meshes/Servo_Horn_v3_6.stl" scale="0.001 0.001 0.001"/>
-    </geometry>
-  </collision>
-</link>
-<link name="Left_Link_v4_1">
-  <inertial>
-    <origin xyz="0.005235109006971023 -0.0028149971111056937 -0.05611727896629981" rpy="0 0 0"/>
-    <mass value="0.12677989413662727"/>
-    <inertia ixx="0.000135" iyy="0.000137" izz="6e-06" ixy="-0.0" iyz="-1e-06" ixz="1e-05"/>
-  </inertial>
-  <visual>
-    <origin xyz="0.165037 -0.115355 -0.017162" rpy="0 0 0"/>
-    <geometry>
-      <mesh filename="file://$(find robot_description)/meshes/Left_Link_v4_1.stl" scale="0.001 0.001 0.001"/>
-    </geometry>
-    <material name="steel_satin"/>
-  </visual>
-  <collision>
-    <origin xyz="0.165037 -0.115355 -0.017162" rpy="0 0 0"/>
-    <geometry>
-      <mesh filename="file://$(find robot_description)/meshes/Left_Link_v4_1.stl" scale="0.001 0.001 0.001"/>
-    </geometry>
-  </collision>
-</link>
-<link name="Foot_v3_1">
-  <inertial>
-    <origin xyz="0.0031275273896734235 -0.005052218921323931 -0.06122868364490067" rpy="0 0 0"/>
-    <mass value="0.31314451205821014"/>
-    <inertia ixx="0.000443" iyy="0.000438" izz="2.5e-05" ixy="-0.0" iyz="0.0" ixz="1e-06"/>
-  </inertial>
-  <visual>
-    <origin xyz="0.162704 -0.115355 0.088726" rpy="0 0 0"/>
-    <geometry>
-      <mesh filename="file://$(find robot_description)/meshes/Foot_v3_1.stl" scale="0.001 0.001 0.001"/>
-    </geometry>
-    <material name="steel_satin"/>
-  </visual>
-  <collision>
-    <origin xyz="0.162704 -0.115355 0.088726" rpy="0 0 0"/>
-    <geometry>
-      <mesh filename="file://$(find robot_description)/meshes/Foot_v3_1.stl" scale="0.001 0.001 0.001"/>
-    </geometry>
-  </collision>
-</link>
-<link name="Left_Link_v4_2">
-  <inertial>
-    <origin xyz="0.005235457637564361 -0.0028148450377657175 -0.056117038923210835" rpy="0 0 0"/>
-    <mass value="0.12677989413662727"/>
-    <inertia ixx="0.000135" iyy="0.000137" izz="6e-06" ixy="-0.0" iyz="-1e-06" ixz="1e-05"/>
-  </inertial>
-  <visual>
-    <origin xyz="-0.143797 -0.115329 -0.017258" rpy="0 0 0"/>
-    <geometry>
-      <mesh filename="file://$(find robot_description)/meshes/Left_Link_v4_2.stl" scale="0.001 0.001 0.001"/>
-    </geometry>
-    <material name="steel_satin"/>
-  </visual>
-  <collision>
-    <origin xyz="-0.143797 -0.115329 -0.017258" rpy="0 0 0"/>
-    <geometry>
-      <mesh filename="file://$(find robot_description)/meshes/Left_Link_v4_2.stl" scale="0.001 0.001 0.001"/>
-    </geometry>
-  </collision>
-</link>
-<link name="Component1_Mirror___4__1">
-  <inertial>
-    <origin xyz="0.005597894046904056 0.002814845037766786 -0.05642367984565573" rpy="0 0 0"/>
-    <mass value="0.1267798941366273"/>
-    <inertia ixx="0.000135" iyy="0.000137" izz="6e-06" ixy="0.0" iyz="1e-06" ixz="1e-05"/>
-  </inertial>
-  <visual>
-    <origin xyz="-0.143797 0.115329 -0.017258" rpy="0 0 0"/>
-    <geometry>
-      <mesh filename="file://$(find robot_description)/meshes/Component1_Mirror___4__1.stl" scale="0.001 0.001 0.001"/>
-    </geometry>
-    <material name="steel_satin"/>
-  </visual>
-  <collision>
-    <origin xyz="-0.143797 0.115329 -0.017258" rpy="0 0 0"/>
-    <geometry>
-      <mesh filename="file://$(find robot_description)/meshes/Component1_Mirror___4__1.stl" scale="0.001 0.001 0.001"/>
-    </geometry>
-  </collision>
-</link>
-<link name="Component1_Mirror___4__2">
-  <inertial>
-    <origin xyz="0.005235109006970551 0.0028149971111054717 -0.05611727896629981" rpy="0 0 0"/>
-    <mass value="0.1267798941366273"/>
-    <inertia ixx="0.000135" iyy="0.000137" izz="6e-06" ixy="0.0" iyz="1e-06" ixz="1e-05"/>
-  </inertial>
-  <visual>
-    <origin xyz="0.165037 0.115355 -0.017162" rpy="0 0 0"/>
-    <geometry>
-      <mesh filename="file://$(find robot_description)/meshes/Component1_Mirror___4__2.stl" scale="0.001 0.001 0.001"/>
-    </geometry>
-    <material name="steel_satin"/>
-  </visual>
-  <collision>
-    <origin xyz="0.165037 0.115355 -0.017162" rpy="0 0 0"/>
-    <geometry>
-      <mesh filename="file://$(find robot_description)/meshes/Component1_Mirror___4__2.stl" scale="0.001 0.001 0.001"/>
-    </geometry>
-  </collision>
-</link>
-<link name="Foot_v3_2">
-  <inertial>
-    <origin xyz="0.0031278760202663736 0.004997933152016104 -0.061228443601811774" rpy="0 0 0"/>
-    <mass value="0.31314451205821014"/>
-    <inertia ixx="0.000443" iyy="0.000438" izz="2.5e-05" ixy="-0.0" iyz="0.0" ixz="1e-06"/>
-  </inertial>
-  <visual>
-    <origin xyz="-0.14613 -0.106349 0.08863" rpy="0 0 0"/>
-    <geometry>
-      <mesh filename="file://$(find robot_description)/meshes/Foot_v3_2.stl" scale="0.001 0.001 0.001"/>
-    </geometry>
-    <material name="steel_satin"/>
-  </visual>
-  <collision>
-    <origin xyz="-0.14613 -0.106349 0.08863" rpy="0 0 0"/>
-    <geometry>
-      <mesh filename="file://$(find robot_description)/meshes/Foot_v3_2.stl" scale="0.001 0.001 0.001"/>
-    </geometry>
-  </collision>
-</link>
-<link name="Mini_Link_v3_3">
-  <inertial>
-    <origin xyz="0.015778623836727845 0.001939671690657202 0.002782107313249153" rpy="0 0 0"/>
-    <mass value="0.01656743535976172"/>
-    <inertia ixx="1e-06" iyy="2e-06" izz="2e-06" ixy="0.0" iyz="0.0" ixz="-0.0"/>
-  </inertial>
-  <visual>
-    <origin xyz="-0.145671 -0.110329 0.007194" rpy="0 0 0"/>
-    <geometry>
-      <mesh filename="file://$(find robot_description)/meshes/Mini_Link_v3_3.stl" scale="0.001 0.001 0.001"/>
-    </geometry>
-    <material name="steel_satin"/>
-  </visual>
-  <collision>
-    <origin xyz="-0.145671 -0.110329 0.007194" rpy="0 0 0"/>
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