Commit message: repalced rviz with foxglove visualization

File: robot_ws/src/robot_desc/urdf/robot_core.xacro (robot description, xacro)
@@ -10,5 +10,5 @@
     <origin xyz="0 0 0" rpy="0 0 0"/>
     <geometry>
-      <mesh filename="file://$(find robot_desc)/urdf/meshes/base_link.stl" scale="0.001 0.001 0.001"/>
+      <mesh filename="package://robot_desc/urdf/meshes/base_link.stl" scale="0.001 0.001 0.001"/>
     </geometry>
   </visual>
@@ -16,5 +16,5 @@
     <origin xyz="0 0 0" rpy="0 0 0"/>
     <geometry>
-      <mesh filename="file://$(find robot_desc)/urdf/meshes/base_link.stl" scale="0.001 0.001 0.001"/>
+      <mesh filename="package://robot_desc/urdf/meshes/base_link.stl" scale="0.001 0.001 0.001"/>
     </geometry>
   </collision>
@@ -29,5 +29,5 @@
     <origin xyz="-0.1184 -0.076 -0.0196" rpy="0 0 0"/>
     <geometry>
-      <mesh filename="file://$(find robot_desc)/urdf/meshes/Right_Front_Leg_Mount_v1_1.stl" scale="0.001 0.001 0.001"/>
+      <mesh filename="package://robot_desc/urdf/meshes/Right_Front_Leg_Mount_v1_1.stl" scale="0.001 0.001 0.001"/>
     </geometry>
   </visual>
@@ -35,5 +35,5 @@
     <origin xyz="-0.1184 -0.076 -0.0196" rpy="0 0 0"/>
     <geometry>
-      <mesh filename="file://$(find robot_desc)/urdf/meshes/Right_Front_Leg_Mount_v1_1.stl" scale="0.001 0.001 0.001"/>
+      <mesh filename="package://robot_desc/urdf/meshes/Right_Front_Leg_Mount_v1_1.stl" scale="0.001 0.001 0.001"/>
     </geometry>
   </collision>
@@ -48,5 +48,5 @@
     <origin xyz="0.1184 -0.076 -0.0196" rpy="0 0 0"/>
     <geometry>
-      <mesh filename="file://$(find robot_desc)/urdf/meshes/Right_Back_Leg_Mount_v1_1.stl" scale="0.001 0.001 0.001"/>
+      <mesh filename="package://robot_desc/urdf/meshes/Right_Back_Leg_Mount_v1_1.stl" scale="0.001 0.001 0.001"/>
     </geometry>
   </visual>
@@ -54,5 +54,5 @@
     <origin xyz="0.1184 -0.076 -0.0196" rpy="0 0 0"/>
     <geometry>
-      <mesh filename="file://$(find robot_desc)/urdf/meshes/Right_Back_Leg_Mount_v1_1.stl" scale="0.001 0.001 0.001"/>
+      <mesh filename="package://robot_desc/urdf/meshes/Right_Back_Leg_Mount_v1_1.stl" scale="0.001 0.001 0.001"/>
     </geometry>
   </collision>
@@ -67,5 +67,5 @@
     <origin xyz="0.1184 0.076 -0.0196" rpy="0 0 0"/>
     <geometry>
-      <mesh filename="file://$(find robot_desc)/urdf/meshes/Left_Back_Leg_Mount_v1_1.stl" scale="0.001 0.001 0.001"/>
+      <mesh filename="package://robot_desc/urdf/meshes/Left_Back_Leg_Mount_v1_1.stl" scale="0.001 0.001 0.001"/>
     </geometry>
   </visual>
@@ -73,5 +73,5 @@
     <origin xyz="0.1184 0.076 -0.0196" rpy="0 0 0"/>
     <geometry>
-      <mesh filename="file://$(find robot_desc)/urdf/meshes/Left_Back_Leg_Mount_v1_1.stl" scale="0.001 0.001 0.001"/>
+      <mesh filename="package://robot_desc/urdf/meshes/Left_Back_Leg_Mount_v1_1.stl" scale="0.001 0.001 0.001"/>
     </geometry>
   </collision>
@@ -86,5 +86,5 @@
     <origin xyz="-0.1184 0.076 -0.0196" rpy="0 0 0"/>
     <geometry>
-      <mesh filename="file://$(find robot_desc)/urdf/meshes/Left_Front_Leg_Mount_v1_1.stl" scale="0.001 0.001 0.001"/>
+      <mesh filename="package://robot_desc/urdf/meshes/Left_Front_Leg_Mount_v1_1.stl" scale="0.001 0.001 0.001"/>
     </geometry>
   </visual>
@@ -92,5 +92,5 @@
     <origin xyz="-0.1184 0.076 -0.0196" rpy="0 0 0"/>
     <geometry>
-      <mesh filename="file://$(find robot_desc)/urdf/meshes/Left_Front_Leg_Mount_v1_1.stl" scale="0.001 0.001 0.001"/>
+      <mesh filename="package://robot_desc/urdf/meshes/Left_Front_Leg_Mount_v1_1.stl" scale="0.001 0.001 0.001"/>
     </geometry>
   </collision>
@@ -105,5 +105,5 @@
     <origin xyz="0.165037 -0.115355 -0.017162" rpy="0 0 0"/>
     <geometry>
-      <mesh filename="file://$(find robot_desc)/urdf/meshes/Left_Link_v4_1.stl" scale="0.001 0.001 0.001"/>
+      <mesh filename="package://robot_desc/urdf/meshes/Left_Link_v4_1.stl" scale="0.001 0.001 0.001"/>
     </geometry>
   </visual>
@@ -111,5 +111,5 @@
     <origin xyz="0.165037 -0.115355 -0.017162" rpy="0 0 0"/>
     <geometry>
-      <mesh filename="file://$(find robot_desc)/urdf/meshes/Left_Link_v4_1.stl" scale="0.001 0.001 0.001"/>
+      <mesh filename="package://robot_desc/urdf/meshes/Left_Link_v4_1.stl" scale="0.001 0.001 0.001"/>
     </geometry>
   </collision>
@@ -124,5 +124,5 @@
     <origin xyz="0.162704 -0.115355 0.088726" rpy="0 0 0"/>
     <geometry>
-      <mesh filename="file://$(find robot_desc)/urdf/meshes/Foot_v3_1.stl" scale="0.001 0.001 0.001"/>
+      <mesh filename="package://robot_desc/urdf/meshes/Foot_v3_1.stl" scale="0.001 0.001 0.001"/>
     </geometry>
   </visual>
@@ -130,5 +130,5 @@
     <origin xyz="0.162704 -0.115355 0.088726" rpy="0 0 0"/>
     <geometry>
-      <mesh filename="file://$(find robot_desc)/urdf/meshes/Foot_v3_1.stl" scale="0.001 0.001 0.001"/>
+      <mesh filename="package://robot_desc/urdf/meshes/Foot_v3_1.stl" scale="0.001 0.001 0.001"/>
     </geometry>
   </collision>
@@ -150,5 +150,5 @@
     <origin xyz="-0.143797 -0.115329 -0.017258" rpy="0 0 0"/>
     <geometry>
-      <mesh filename="file://$(find robot_desc)/urdf/meshes/Left_Link_v4_2.stl" scale="0.001 0.001 0.001"/>
+      <mesh filename="package://robot_desc/urdf/meshes/Left_Link_v4_2.stl" scale="0.001 0.001 0.001"/>
     </geometry>
   </visual>
@@ -156,5 +156,5 @@
     <origin xyz="-0.143797 -0.115329 -0.017258" rpy="0 0 0"/>
     <geometry>
-      <mesh filename="file://$(find robot_desc)/urdf/meshes/Left_Link_v4_2.stl" scale="0.001 0.001 0.001"/>
+      <mesh filename="package://robot_desc/urdf/meshes/Left_Link_v4_2.stl" scale="0.001 0.001 0.001"/>
     </geometry>
   </collision>
@@ -169,5 +169,5 @@
     <origin xyz="-0.143797 0.115329 -0.017258" rpy="0 0 0"/>
     <geometry>
-      <mesh filename="file://$(find robot_desc)/urdf/meshes/Component1_Mirror___4__1.stl" scale="0.001 0.001 0.001"/>
+      <mesh filename="package://robot_desc/urdf/meshes/Component1_Mirror___4__1.stl" scale="0.001 0.001 0.001"/>
     </geometry>
   </visual>
@@ -175,5 +175,5 @@
     <origin xyz="-0.143797 0.115329 -0.017258" rpy="0 0 0"/>
     <geometry>
-      <mesh filename="file://$(find robot_desc)/urdf/meshes/Component1_Mirror___4__1.stl" scale="0.001 0.001 0.001"/>
+      <mesh filename="package://robot_desc/urdf/meshes/Component1_Mirror___4__1.stl" scale="0.001 0.001 0.001"/>
     </geometry>
   </collision>
@@ -188,5 +188,5 @@
     <origin xyz="0.165037 0.115355 -0.017162" rpy="0 0 0"/>
     <geometry>
-      <mesh filename="file://$(find robot_desc)/urdf/meshes/Component1_Mirror___4__2.stl" scale="0.001 0.001 0.001"/>
+      <mesh filename="package://robot_desc/urdf/meshes/Component1_Mirror___4__2.stl" scale="0.001 0.001 0.001"/>
     </geometry>
   </visual>
@@ -194,5 +194,5 @@
     <origin xyz="0.165037 0.115355 -0.017162" rpy="0 0 0"/>
     <geometry>
-      <mesh filename="file://$(find robot_desc)/urdf/meshes/Component1_Mirror___4__2.stl" scale="0.001 0.001 0.001"/>
+      <mesh filename="package://robot_desc/urdf/meshes/Component1_Mirror___4__2.stl" scale="0.001 0.001 0.001"/>
     </geometry>
   </collision>
@@ -207,5 +207,5 @@
     <origin xyz="-0.14613 -0.106349 0.08863" rpy="0 0 0"/>
     <geometry>
-      <mesh filename="file://$(find robot_desc)/urdf/meshes/Foot_v3_2.stl" scale="0.001 0.001 0.001"/>
+      <mesh filename="package://robot_desc/urdf/meshes/Foot_v3_2.stl" scale="0.001 0.001 0.001"/>
     </geometry>
   </visual>
@@ -213,5 +213,5 @@
     <origin xyz="-0.14613 -0.106349 0.08863" rpy="0 0 0"/>
     <geometry>
-      <mesh filename="file://$(find robot_desc)/urdf/meshes/Foot_v3_2.stl" scale="0.001 0.001 0.001"/>
+      <mesh filename="package://robot_desc/urdf/meshes/Foot_v3_2.stl" scale="0.001 0.001 0.001"/>
     </geometry>
   </collision>
@@ -233,5 +233,5 @@
     <origin xyz="0.162704 0.115355 0.088726" rpy="0 0 0"/>
     <geometry>
-      <mesh filename="file://$(find robot_desc)/urdf/meshes/Component1_Mirror___5__2.stl" scale="0.001 0.001 0.001"/>
+      <mesh filename="package://robot_desc/urdf/meshes/Component1_Mirror___5__2.stl" scale="0.001 0.001 0.001"/>
     </geometry>
   </visual>
@@ -239,5 +239,5 @@
     <origin xyz="0.162704 0.115355 0.088726" rpy="0 0 0"/>
     <geometry>
-      <mesh filename="file://$(find robot_desc)/urdf/meshes/Component1_Mirror___5__2.stl" scale="0.001 0.001 0.001"/>
+      <mesh filename="package://robot_desc/urdf/meshes/Component1_Mirror___5__2.stl" scale="0.001 0.001 0.001"/>
     </geometry>
   </collision>
@@ -259,5 +259,5 @@
     <origin xyz="-0.146492 0.115329 0.088937" rpy="0 0 0"/>
     <geometry>
-      <mesh filename="file://$(find robot_desc)/urdf/meshes/Component1_Mirror___5__1.stl" scale="0.001 0.001 0.001"/>
+      <mesh filename="package://robot_desc/urdf/meshes/Component1_Mirror___5__1.stl" scale="0.001 0.001 0.001"/>
     </geometry>
   </visual>
@@ -265,5 +265,5 @@
     <origin xyz="-0.146492 0.115329 0.088937" rpy="0 0 0"/>
     <geometry>
-      <mesh filename="file://$(find robot_desc)/urdf/meshes/Component1_Mirror___5__1.stl" scale="0.001 0.001 0.001"/>
+      <mesh filename="package://robot_desc/urdf/meshes/Component1_Mirror___5__1.stl" scale="0.001 0.001 0.001"/>
     </geometry>
   </collision>

Commit message: Updated joint limits in urdf files

File: robot_ws/src/robot_desc/urdf/robot_core.xacro (robot description, xacro)
@@ -281,5 +281,5 @@
   <child link="Right_Front_Leg_Mount_v1_1"/>
   <axis xyz="1.0 0.0 -0.0"/>
-  <limit upper="1.570796" lower="-1.570796" effort="10000" velocity="100"/>
+  <limit upper="3.14159" lower="-3.14159" effort="10000" velocity="100"/>
 </joint>
 <joint name="Revolute_3" type="revolute">
@@ -288,5 +288,5 @@
   <child link="Right_Back_Leg_Mount_v1_1"/>
   <axis xyz="-1.0 -0.0 0.0"/>
-  <limit upper="1.570796" lower="-1.570796" effort="10000" velocity="100"/>
+  <limit upper="3.14159" lower="-3.14159" effort="10000" velocity="100"/>
 </joint>
 <joint name="Revolute_4" type="revolute">
@@ -295,5 +295,5 @@
   <child link="Left_Back_Leg_Mount_v1_1"/>
   <axis xyz="-1.0 -0.0 0.0"/>
-  <limit upper="1.570796" lower="-1.570796" effort="10000" velocity="100"/>
+  <limit upper="3.14159" lower="-3.14159" effort="10000" velocity="100"/>
 </joint>
 <joint name="Revolute_5" type="revolute">
@@ -302,5 +302,5 @@
   <child link="Left_Front_Leg_Mount_v1_1"/>
   <axis xyz="1.0 0.0 -0.0"/>
-  <limit upper="1.570796" lower="-1.570796" effort="10000" velocity="100"/>
+  <limit upper="3.14159" lower="-3.14159" effort="10000" velocity="100"/>
 </joint>
 <joint name="Revolute_20" type="revolute">
@@ -309,5 +309,5 @@
   <child link="Left_Link_v4_1"/>
   <axis xyz="-0.0 -1.0 -0.0"/>
-  <limit upper="1.570796" lower="-1.570796" effort="10000" velocity="100"/>
+  <limit upper="3.14159" lower="-3.14159" effort="10000" velocity="100"/>
 </joint>
 <joint name="Revolute_23" type="revolute">
@@ -316,5 +316,5 @@
   <child link="Foot_v3_1"/>
   <axis xyz="0.0 1.0 0.0"/>
-  <limit upper="1.570796" lower="-1.570796" effort="10000" velocity="100"/>
+  <limit upper="3.14159" lower="-3.14159" effort="10000" velocity="100"/>
 </joint>
 <joint name="Revolute_25" type="revolute">
@@ -323,5 +323,5 @@
   <child link="Left_Link_v4_2"/>
   <axis xyz="-0.0 -1.0 -0.0"/>
-  <limit upper="1.570796" lower="-1.570796" effort="10000" velocity="100"/>
+  <limit upper="3.14159" lower="-3.14159" effort="10000" velocity="100"/>
 </joint>
 <joint name="Revolute_31" type="revolute">
@@ -330,5 +330,5 @@
   <child link="Component1_Mirror___4__1"/>
   <axis xyz="-0.0 1.0 0.0"/>
-  <limit upper="1.570796" lower="-1.570796" effort="10000" velocity="100"/>
+  <limit upper="3.14159" lower="-3.14159" effort="10000" velocity="100"/>
 </joint>
 <joint name="Revolute_35" type="revolute">
@@ -337,5 +337,5 @@
   <child link="Component1_Mirror___4__2"/>
   <axis xyz="-0.0 1.0 0.0"/>
-  <limit upper="1.570796" lower="-1.570796" effort="10000" velocity="100"/>
+  <limit upper="3.14159" lower="-3.14159" effort="10000" velocity="100"/>
 </joint>
 <joint name="Revolute_40" type="revolute">
@@ -344,5 +344,5 @@
   <child link="Foot_v3_2"/>
   <axis xyz="0.0 1.0 0.0"/>
-  <limit upper="1.570796" lower="-1.570796" effort="10000" velocity="100"/>
+  <limit upper="3.14159" lower="-3.14159" effort="10000" velocity="100"/>
 </joint>
 <joint name="Revolute_45" type="revolute">
@@ -351,5 +351,5 @@
   <child link="Component1_Mirror___5__2"/>
   <axis xyz="0.0 -1.0 0.0"/>
-  <limit upper="1.570796" lower="-1.570796" effort="10000" velocity="100"/>
+  <limit upper="3.14159" lower="-3.14159" effort="10000" velocity="100"/>
 </joint>
 <joint name="Revolute_48" type="revolute">
@@ -358,5 +358,5 @@
   <child link="Component1_Mirror___5__1"/>
   <axis xyz="-0.0 1.0 0.0"/>
-  <limit upper="1.570796" lower="-1.570796" effort="10000" velocity="100"/>
+  <limit upper="3.14159" lower="-3.14159" effort="10000" velocity="100"/>
 </joint>
 </robot>

File: robot_ws/src/robot_simulation/urdf/robot_core.xacro (robot description, xacro)
@@ -281,5 +281,5 @@
   <child link="Right_Front_Leg_Mount_v1_1"/>
   <axis xyz="1.0 0.0 -0.0"/>
-  <limit upper="1.570796" lower="-1.570796" effort="10000" velocity="100"/>
+  <limit upper="3.14159" lower="-3.14159" effort="10000" velocity="100"/>
 </joint>
 <joint name="Revolute_3" type="revolute">
@@ -288,5 +288,5 @@
   <child link="Right_Back_Leg_Mount_v1_1"/>
   <axis xyz="-1.0 -0.0 0.0"/>
-  <limit upper="1.570796" lower="-1.570796" effort="10000" velocity="100"/>
+  <limit upper="3.14159" lower="-3.14159" effort="10000" velocity="100"/>
 </joint>
 <joint name="Revolute_4" type="revolute">
@@ -295,5 +295,5 @@
   <child link="Left_Back_Leg_Mount_v1_1"/>
   <axis xyz="-1.0 -0.0 0.0"/>
-  <limit upper="1.570796" lower="-1.570796" effort="10000" velocity="100"/>
+  <limit upper="3.14159" lower="-3.14159" effort="10000" velocity="100"/>
 </joint>
 <joint name="Revolute_5" type="revolute">
@@ -302,5 +302,5 @@
   <child link="Left_Front_Leg_Mount_v1_1"/>
   <axis xyz="1.0 0.0 -0.0"/>
-  <limit upper="1.570796" lower="-1.570796" effort="10000" velocity="100"/>
+  <limit upper="3.14159" lower="-3.14159" effort="10000" velocity="100"/>
 </joint>
 <joint name="Revolute_20" type="revolute">
@@ -309,5 +309,5 @@
   <child link="Left_Link_v4_1"/>
   <axis xyz="-0.0 -1.0 -0.0"/>
-  <limit upper="1.570796" lower="-1.570796" effort="10000" velocity="100"/>
+  <limit upper="3.14159" lower="-3.14159" effort="10000" velocity="100"/>
 </joint>
 <joint name="Revolute_23" type="revolute">
@@ -316,5 +316,5 @@
   <child link="Foot_v3_1"/>
   <axis xyz="0.0 1.0 0.0"/>
-  <limit upper="1.570796" lower="-1.570796" effort="10000" velocity="100"/>
+  <limit upper="3.14159" lower="-3.14159" effort="10000" velocity="100"/>
 </joint>
 <joint name="Revolute_25" type="revolute">
@@ -323,5 +323,5 @@
   <child link="Left_Link_v4_2"/>
   <axis xyz="-0.0 -1.0 -0.0"/>
-  <limit upper="1.570796" lower="-1.570796" effort="10000" velocity="100"/>
+  <limit upper="3.14159" lower="-3.14159" effort="10000" velocity="100"/>
 </joint>
 <joint name="Revolute_31" type="revolute">
@@ -330,5 +330,5 @@
   <child link="Component1_Mirror___4__1"/>
   <axis xyz="-0.0 1.0 0.0"/>
-  <limit upper="1.570796" lower="-1.570796" effort="10000" velocity="100"/>
+  <limit upper="3.14159" lower="-3.14159" effort="10000" velocity="100"/>
 </joint>
 <joint name="Revolute_35" type="revolute">
@@ -337,5 +337,5 @@
   <child link="Component1_Mirror___4__2"/>
   <axis xyz="-0.0 1.0 0.0"/>
-  <limit upper="1.570796" lower="-1.570796" effort="10000" velocity="100"/>
+  <limit upper="3.14159" lower="-3.14159" effort="10000" velocity="100"/>
 </joint>
 <joint name="Revolute_40" type="revolute">
@@ -344,5 +344,5 @@
   <child link="Foot_v3_2"/>
   <axis xyz="0.0 1.0 0.0"/>
-  <limit upper="1.570796" lower="-1.570796" effort="10000" velocity="100"/>
+  <limit upper="3.14159" lower="-3.14159" effort="10000" velocity="100"/>
 </joint>
 <joint name="Revolute_45" type="revolute">
@@ -351,5 +351,5 @@
   <child link="Component1_Mirror___5__2"/>
   <axis xyz="0.0 -1.0 0.0"/>
-  <limit upper="1.570796" lower="-1.570796" effort="10000" velocity="100"/>
+  <limit upper="3.14159" lower="-3.14159" effort="10000" velocity="100"/>
 </joint>
 <joint name="Revolute_48" type="revolute">
@@ -358,5 +358,5 @@
   <child link="Component1_Mirror___5__1"/>
   <axis xyz="-0.0 1.0 0.0"/>
-  <limit upper="1.570796" lower="-1.570796" effort="10000" velocity="100"/>
+  <limit upper="3.14159" lower="-3.14159" effort="10000" velocity="100"/>
 </joint>
 </robot>
